File: freeDSP-aurora-extension-i2C-mod-display.kicad_pcb (KiCad board)
At the start: 2 copper layers, 76.1 x 47.1 mm, 10 parts, among them J1 PinHeader_1x04_P2.54mm_Vertic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, J2 PinSocket_1x07_P2.54mm_Vertic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

Commit message: Rev 1.2
Update silkscreen
Parts:
- C1: value 4µ7 -> 4u7
Other:
- board text added: "Vcc (3V3)"
- board text added: "cw 2022 - v1.2"
- board text removed: "Vcc 3V3"
- board text removed: "cw 2022 - v1.1"
Changed lines of the file:
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@@
-(kicad_pcb (version 20220211) (generator pcbnew)
+(kicad_pcb (version 20220308) (generator pcbnew)
   (general
     (thickness 1.6)
@@
   (title_block
     (title "Aurora Display Extension Board (I^{2}C mod)")
-    (date "2022-02-20")
-    (rev "v1.1")
+    (date "2022-04-06")
+    (rev "v1.2")
     (company "cw")
   )
@@
         (effects (font (size 1 1) (thickness 0.15)))
     )
-    (fp_text value "4µ7" (at 1.25 6.25) (layer "F.SilkS")
+    (fp_text value "4u7" (at 1.25 6.25) (layer "F.SilkS")
         (effects (font (size 1 1) (thickness 0.15)))
     )
@@
   (gr_line (start 174.355 75.057) (end 174.355 122.174)
     (stroke (width 0.1) (type solid)) (layer "Edge.Cuts"))
-  (gr_text "cw 2022 - v1.1" (at 136.33 120.252244) (layer "B.Cu")
+  (gr_text "cw 2022 - v1.2" (at 136.33 120.252244) (layer "B.Cu")
     (effects (font (size 1 1) (thickness 0.1)) (justify mirror))
   )
@@
     (effects (font (size 1.6 1.6) (thickness 0.3) bold) (justify left))
   )
-  (gr_text "Vcc 3V3" (at 163.957 104.14) (layer "F.SilkS")
+  (gr_text "Vcc (3V3)" (at 163.957 104.14) (layer "F.SilkS")
     (effects (font (size 1 1) (thickness 0.15)) (justify right))
   )
