File: freeDSP-aurora-extension-i2C-mod-display.kicad_sch (KiCad schematic)
At the start: 4 parts, among them J1 Conn_01x04_Male, J2 Conn_01x07_Female

Commit message: Rev 1.2
Update silkscreen
Changed lines of the file:
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@@
-(kicad_sch (version 20220126) (generator eeschema)
+(kicad_sch (version 20220331) (generator eeschema)
   (paper "A4")
   (title_block
     (title "freeDSP aurora display extension board (I2C mod)")
-    (date "2022-01-22")
-    (rev "v1.1")
+    (date "2022-04-06")
+    (rev "v1.2")
     (company "Carsten Witt (cw)")
     (comment 3 "freeDSP aurora display extension board (I2C mod)")
@@
     (effects (font (size 1.27 1.27)) (justify left bottom))
   )
-  (label "Vcc 3V3" (at 109.22 91.44 0) (fields_autoplaced)
+  (label "Vcc (3V3)" (at 109.22 91.44 0) (fields_autoplaced)
     (effects (font (size 1.27 1.27)) (justify left bottom))
   )
